File: elec/test1/test1.sch (KiCad schematic (older format))
At the start: 7 parts, among them CN10 Conn_02x19_Odd_Even, CN7 Conn_02x19_Odd_Even, J1 Conn_01x04, M1 Motor_DC, U2 L298HN

Commit message: pcb
Parts:
- removed M1: Motor_DC, symbol Motor:Motor_DC
- added J2, J3: Screw_Terminal_01x02, TerminalBlock_MetzConnect:TerminalBlock_MetzConnect_Type011_RT05502HBWC_1x02_P5.00mm_Horizontal, symbol Connector:Screw_Terminal_01x02
Connections:
- net +12V: now also J3.1 (Pin_1)
- net +5V: no longer U2.9 (Vss)
- net GND: now also CN7.22 (Pin_22), J3.2 (Pin_2); no longer CN7.20 (Pin_20)
- net +3V3: now reaches CN7.16 (Pin_16)
- net +3V3: now also U2.9 (Vss)
- net at U2.2 (OUT1): now also J2.1 (Pin_1)
- net at U2.3 (OUT2): now also J2.2 (Pin_2)
Changed lines of the file:
@@
 enc_b
-$Comp
-L power:+5V #PWR0104
-U 1 1 60AF2D4F
-P 9650 2250
-F 0 "#PWR0104" H 9650 2100 50  0001 C CNN
-F 1 "+5V" V 9665 2378 50  0000 L CNN
-F 2 "" H 9650 2250 50  0001 C CNN
-F 3 "" H 9650 2250 50  0001 C CNN
-	1    9650 2250
-	0    1    1    0
-$EndComp
 $Comp
 L Device:R R1
@@
 $EndComp
 $Comp
-L power:+5V #PWR0107
-U 1 1 60AA623E
-P 3950 1200
-F 0 "#PWR0107" H 3950 1050 50  0001 C CNN
-F 1 "+5V" V 3965 1328 50  0000 L CNN
-F 2 "" H 3950 1200 50  0001 C CNN
-F 3 "" H 3950 1200 50  0001 C CNN
-	1    3950 1200
-	1    0    0    -1
-$EndComp
-$Comp
 L power:+12V #PWR0108
 U 1 1 60AA672B
@@
 Wire Wire Line
 	3350 1600 2800 1600
-Wire Wire Line
-	4550 1700 4900 1700
-Wire Wire Line
-	4550 1800 4900 1800
 $Comp
 L power:GND #PWR0106
@@
 	1    0    0    -1
 $EndComp
-$Comp
-L Motor:Motor_DC M1
-U 1 1 60AA92CB
-P 5250 1700
-F 0 "M1" H 5408 1696 50  0000 L CNN
-F 1 "Motor_DC" H 5408 1605 50  0000 L CNN
-F 2 "" H 5250 1610 50  0001 C CNN
-F 3 "~" H 5250 1610 50  0001 C CNN
-	1    5250 1700
-	1    0    0    -1
-$EndComp
-Wire Wire Line
-	5250 1500 4900 1500
-Wire Wire Line
-	4900 1500 4900 1700
-Wire Wire Line
-	5250 2000 4900 2000
-Wire Wire Line
-	4900 2000 4900 1800
 Text Label 2800 1400 0    50   ~ 0
 motor_ina
@@
 NoConn ~ 3350 1900
 NoConn ~ 3350 2000
-Wire Wire Line
-	9650 2250 9550 2250
-$Comp
-L power:GND #PWR0105
-U 1 1 60AF2ED0
-P 9650 2350
-F 0 "#PWR0105" H 9650 2100 50  0001 C CNN
-F 1 "GND" V 9655 2222 50  0000 R CNN
-F 2 "" H 9650 2350 50  0001 C CNN
-F 3 "" H 9650 2350 50  0001 C CNN
-	1    9650 2350
-	0    -1   -1   0
-$EndComp
-Wire Wire Line
-	9650 2350 9550 2350
-Connection ~ 9650 2250
-$Comp
-L power:PWR_FLAG #FLG0101
-U 1 1 60A9CCD6
-P 9650 2250
-F 0 "#FLG0101" H 9650 2325 50  0001 C CNN
-F 1 "PWR_FLAG" H 9800 2400 50  0000 C CNN
-F 2 "" H 9650 2250 50  0001 C CNN
-F 3 "~" H 9650 2250 50  0001 C CNN
-	1    9650 2250
-	1    0    0    -1
-$EndComp
-$Comp
-L power:PWR_FLAG #FLG0102
-U 1 1 60AA2F94
-P 9650 2350
-F 0 "#FLG0102" H 9650 2425 50  0001 C CNN
-F 1 "PWR_FLAG" H 9500 2500 50  0000 C CNN
-F 2 "" H 9650 2350 50  0001 C CNN
-F 3 "~" H 9650 2350 50  0001 C CNN
-	1    9650 2350
-	-1   0    0    1
-$EndComp
 $Comp
 L Connector_Generic:Conn_02x19_Odd_Even CN7
@@
 	1    0    0    -1
 $EndComp
-Connection ~ 9650 2350
+$Comp
+L Connector:Screw_Terminal_01x02 J2
+U 1 1 60AC0B5D
+P 4800 1700
+F 0 "J2" H 4880 1692 50  0000 L CNN
+F 1 "Screw_Terminal_01x02" H 4880 1601 50  0000 L CNN
+F 2 "TerminalBlock_MetzConnect:TerminalBlock_MetzConnect_Type011_RT05502HBWC_1x02_P5.00mm_Horizontal" H 4800 1700 50  0001 C CNN
+F 3 "~" H 4800 1700 50  0001 C CNN
+	1    4800 1700
+	1    0    0    -1
+$EndComp
+Wire Wire Line
+	4600 1700 4550 1700
+Wire Wire Line
+	4600 1800 4550 1800
+$Comp
+L power:+3.3V #PWR0107
+U 1 1 60AD8902
+P 3950 1200
+F 0 "#PWR0107" H 3950 1050 50  0001 C CNN
+F 1 "+3.3V" V 3950 1400 50  0000 C CNN
+F 2 "" H 3950 1200 50  0001 C CNN
+F 3 "" H 3950 1200 50  0001 C CNN
+	1    3950 1200
+	1    0    0    -1
+$EndComp
+$Comp
+L power:+12V #PWR0109
+U 1 1 60ACAF17
+P 5400 1050
+F 0 "#PWR0109" H 5400 900 50  0001 C CNN
+F 1 "+12V" V 5400 1250 50  0000 C CNN
+F 2 "" H 5400 1050 50  0001 C CNN
+F 3 "" H 5400 1050 50  0001 C CNN
+	1    5400 1050
+	0    1    1    0
+$EndComp
+$Comp
+L power:+5V #PWR0104
+U 1 1 60AF2D4F
+P 9700 2250
+F 0 "#PWR0104" H 9700 2100 50  0001 C CNN
+F 1 "+5V" V 9715 2378 50  0000 L CNN
+F 2 "" H 9700 2250 50  0001 C CNN
+F 3 "" H 9700 2250 50  0001 C CNN
+	1    9700 2250
+	0    1    1    0
+$EndComp
+$Comp
+L Connector:Screw_Terminal_01x02 J3
+U 1 1 60AC923C
+P 5200 1050
+F 0 "J3" H 5280 1042 50  0000 L CNN
+F 1 "Screw_Terminal_01x02" H 5280 951 50  0000 L CNN
+F 2 "TerminalBlock_MetzConnect:TerminalBlock_MetzConnect_Type011_RT05502HBWC_1x02_P5.00mm_Horizontal" H 5200 1050 50  0001 C CNN
+F 3 "~" H 5200 1050 50  0001 C CNN
+	1    5200 1050
+	-1   0    0    1
+$EndComp
+$Comp
+L power:GND #PWR0110
+U 1 1 60ACB4F5
+P 5400 950
+F 0 "#PWR0110" H 5400 700 50  0001 C CNN
+F 1 "GND" H 5405 777 50  0000 C CNN
+F 2 "" H 5400 950 50  0001 C CNN
+F 3 "" H 5400 950 50  0001 C CNN
+	1    5400 950
+	0    -1   -1   0
+$EndComp
+$Comp
+L power:+3.3V #PWR0111
+U 1 1 60AED464
+P 9700 2150
+F 0 "#PWR0111" H 9700 2000 50  0001 C CNN
+F 1 "+3.3V" V 9700 2350 50  0000 C CNN
+F 2 "" H 9700 2150 50  0001 C CNN
+F 3 "" H 9700 2150 50  0001 C CNN
+	1    9700 2150
+	0    1    1    0
+$EndComp
+$Comp
+L power:PWR_FLAG #FLG0101
+U 1 1 60A9CCD6
+P 9700 2250
+F 0 "#FLG0101" H 9700 2325 50  0001 C CNN
+F 1 "PWR_FLAG" H 9700 2400 50  0000 C CNN
+F 2 "" H 9700 2250 50  0001 C CNN
+F 3 "~" H 9700 2250 50  0001 C CNN
+	1    9700 2250
+	-1   0    0    1
+$EndComp
+Wire Wire Line
+	9700 2150 9550 2150
+$Comp
+L power:PWR_FLAG #FLG0102
+U 1 1 60B02081
+P 9700 2150
+F 0 "#FLG0102" H 9700 2225 50  0001 C CNN
+F 1 "PWR_FLAG" H 9700 2300 50  0000 C CNN
+F 2 "" H 9700 2150 50  0001 C CNN
+F 3 "~" H 9700 2150 50  0001 C CNN
+	1    9700 2150
+	1    0    0    -1
+$EndComp
+Connection ~ 9700 2150
+Wire Wire Line
+	9550 2250 9700 2250
+Connection ~ 9700 2250
+Wire Wire Line
+	9550 2450 9800 2450
+$Comp
+L power:GND #PWR0105
+U 1 1 60AF2ED0
+P 9800 2450
+F 0 "#PWR0105" H 9800 2200 50  0001 C CNN
+F 1 "GND" V 9805 2322 50  0000 R CNN
+F 2 "" H 9800 2450 50  0001 C CNN
+F 3 "" H 9800 2450 50  0001 C CNN
+	1    9800 2450
+	1    0    0    -1
+$EndComp
+$Comp
+L power:PWR_FLAG #FLG0103
+U 1 1 60B17C1E
+P 5400 1050
+F 0 "#FLG0103" H 5400 1125 50  0001 C CNN
+F 1 "PWR_FLAG" H 5400 1200 50  0000 C CNN
+F 2 "" H 5400 1050 50  0001 C CNN
+F 3 "~" H 5400 1050 50  0001 C CNN
+	1    5400 1050
+	-1   0    0    1
+$EndComp
 $EndSCHEMATC

Commit message: regualator
Parts:
- added C1, C2: C 3.3uf, symbol Device:C
- added C3, C4: C 0.1uF, symbol Device:C
- added D1, D2: LED, symbol Device:LED
- added D3, D4, D5, D6: 1N4007, Diode_THT:D_DO-41_SOD81_P10.16mm_Horizontal, symbol Diode:1N4007
- added R100: R, symbol Device:R
- added U1: LM7805_TO220, Package_TO_SOT_THT:TO-220-3_Vertical, symbol Regulator_Linear:LM7805_TO220
- added U3: LP2950-3.3_TO92, Package_TO_SOT_THT:TO-92_Inline, symbol Regulator_Linear:LP2950-3.3_TO92
Connections:
- net +12V: now also CN7.24 (Pin_24), C1.1, D3.1 (K), D5.1 (K), U1.1 (VI)
- net +3V3: now also C4.1, D2.2 (A), U3.1 (VO); no longer CN7.16 (Pin_16)
- net +5V: now also C2.1, C3.1, D1.2 (A), U1.3 (VO), U3.3 (VI); no longer CN7.18 (Pin_18)
- net GND: now also U2.1 (SENSE_A), U2.15 (SENSE_B), C1.2, C2.2, C3.2, C4.2, D2.1 (K), D4.2 (A), D6.2 (A), R100.1, U1.2 (GND), U3.2 (GND)
- net at J2.1 (Pin_1), U2.2 (OUT1): now also D3.2 (A), D4.1 (K)
- net at J2.2 (Pin_2), U2.3 (OUT2): now also D5.2 (A), D6.1 (K)
- new net: D1.1 (K), R100.2
- no-connect marks 7 -> 5
Other:
- note added: "REGULATOR\n"
- moved on the sheet: J1, J2, J3, R1, R2, U2

Commit message: new_pin_config
Parts:
- added J4: Conn_01x04, Connector_JST:JST_XH_S4B-XH-A-1_1x04_P2.50mm_Horizontal, symbol Connector_Generic:Conn_01x04
- added J5: Conn_01x02, Connector_JST:JST_XH_S2B-XH-A_1x02_P2.50mm_Horizontal, symbol Connector_Generic:Conn_01x02
Connections:
- net +12V: now also J4.1 (Pin_1)
- net +5V: now also U2.6 (EnA)
- net GND: now also J4.4 (Pin_4), J5.2 (Pin_2)
- net motor_pwm2: now reaches CN10.15 (Pin_15)
- net motor_pwm2: now also U2.7 (IN2)
- net limit_switch: now reaches CN10.19 (Pin_19)
- net limit_switch: now also J5.1 (Pin_1)
- net I2C_SCL: now reaches CN10.3 (Pin_3)
- net I2C_SCL: now also J4.2 (Pin_2)
- net I2C_SDA: now reaches CN10.5 (Pin_5)
- net I2C_SDA: now also J4.3 (Pin_3)
- net motor_ina: no longer names the net of CN10.2 (Pin_2)
- net motor_ina: no longer U2.5 (IN1)
- net motor_inb: no longer names the net of CN10.1 (Pin_1)
- net motor_inb: no longer U2.7 (IN2)
- net motro_pwm renamed motor_pwm1
- net motor_pwm1: now also U2.5 (IN1); no longer U2.6 (EnA)
Other:
- note added: "END EFFECTOR"
- note added: "LIMIT SWITCH\n"
Changed lines of the file:
@@
 $EndComp
 Text Label 850  1450 0    50   ~ 0
-motor_ina
+motor_pwm1
 Text Label 850  1550 0    50   ~ 0
-motor_inb
-Text Label 850  1650 0    50   ~ 0
-motro_pwm
+motor_pwm2
 Text Notes 3850 4650 0    50   ~ 0
 *enc_a,enc_b to nucleo
@@
 Text Notes 850  900  0    98   ~ 0
 MOTOR DRIVER\n
-Text Label 10800 1450 0    50   ~ 0
-motor_ina
-Text Label 10300 1450 2    50   ~ 0
-motor_inb
 Text Label 10300 2050 2    50   ~ 0
-motro_pwm
+motor_pwm1
 Wire Notes Line
 	3350 3350 3350 4750
@@
 Wire Wire Line
 	1800 2650 1850 2650
-Wire Wire Line
-	1400 1650 850  1650
 Wire Wire Line
 	1400 1550 850  1550
@@
 Wire Wire Line
 	2450 4400 2650 4400
+Text Label 10300 2150 2    50   ~ 0
+motor_pwm2
+$Comp
+L power:+5V #PWR0119
+U 1 1 60E31E2A
+P 1400 1650
+F 0 "#PWR0119" H 1400 1500 50  0001 C CNN
+F 1 "+5V" V 1415 1778 50  0000 L CNN
+F 2 "" H 1400 1650 50  0001 C CNN
+F 3 "" H 1400 1650 50  0001 C CNN
+	1    1400 1650
+	0    -1   -1   0
+$EndComp
+Text Label 10300 2350 2    50   ~ 0
+limit_switch
+Text Label 10300 1550 2    50   ~ 0
+I2C_SCL
+Text Label 10300 1650 2    50   ~ 0
+I2C_SDA
+$Comp
+L Connector_Generic:Conn_01x04 J4
+U 1 1 60E366CD
+P 5900 1250
+F 0 "J4" H 5980 1242 50  0000 L CNN
+F 1 "Conn_01x04" H 5980 1151 50  0000 L CNN
+F 2 "Connector_JST:JST_XH_S4B-XH-A-1_1x04_P2.50mm_Horizontal" H 5900 1250 50  0001 C CNN
+F 3 "~" H 5900 1250 50  0001 C CNN
+	1    5900 1250
+	1    0    0    -1
+$EndComp
+$Comp
+L power:+12V #PWR0120
+U 1 1 60E38079
+P 5700 1150
+F 0 "#PWR0120" H 5700 1000 50  0001 C CNN
+F 1 "+12V" V 5700 1350 50  0000 C CNN
+F 2 "" H 5700 1150 50  0001 C CNN
+F 3 "" H 5700 1150 50  0001 C CNN
+	1    5700 1150
+	0    -1   -1   0
+$EndComp
+$Comp
+L power:GND #PWR0121
+U 1 1 60E39E68
+P 5700 1450
+F 0 "#PWR0121" H 5700 1200 50  0001 C CNN
+F 1 "GND" H 5705 1277 50  0000 C CNN
+F 2 "" H 5700 1450 50  0001 C CNN
+F 3 "" H 5700 1450 50  0001 C CNN
+	1    5700 1450
+	0    1    1    0
+$EndComp
+Text Label 5550 1250 2    50   ~ 0
+I2C_SCL
+Text Label 5550 1350 2    50   ~ 0
+I2C_SDA
+Wire Wire Line
+	5700 1250 5550 1250
+Wire Wire Line
+	5700 1350 5550 1350
+$Comp
+L Connector_Generic:Conn_01x02 J5
+U 1 1 60E43733
+P 5950 2700
+F 0 "J5" H 6030 2692 50  0000 L CNN
+F 1 "Conn_01x02" H 6030 2601 50  0000 L CNN
+F 2 "Connector_JST:JST_XH_S2B-XH-A_1x02_P2.50mm_Horizontal" H 5950 2700 50  0001 C CNN
+F 3 "~" H 5950 2700 50  0001 C CNN
+	1    5950 2700
+	1    0    0    -1
+$EndComp
+Text Label 5600 2700 2    50   ~ 0
+limit_switch
+Wire Wire Line
+	5750 2700 5600 2700
+$Comp
+L power:GND #PWR0122
+U 1 1 60E47EFB
+P 5750 2800
+F 0 "#PWR0122" H 5750 2550 50  0001 C CNN
+F 1 "GND" H 5755 2627 50  0000 C CNN
+F 2 "" H 5750 2800 50  0001 C CNN
+F 3 "" H 5750 2800 50  0001 C CNN
+	1    5750 2800
+	0    1    1    0
+$EndComp
+Text Notes 4800 950  0    98   ~ 0
+END EFFECTOR
+Text Notes 4750 2450 0    98   ~ 0
+LIMIT SWITCH\n
+Wire Notes Line
+	4650 1700 6600 1700
+Wire Notes Line
+	6600 1700 6600 700
+Wire Notes Line
+	6600 700  4650 700
+Wire Notes Line
+	4650 3150 6650 3150
+Wire Notes Line
+	6650 3150 6650 2050
+Wire Notes Line
+	6650 2050 4650 2050
+Wire Notes Line
+	4650 2050 4650 3150
+Wire Notes Line
+	4650 700  4650 1700
 $EndSCHEMATC

Commit message: pcb_V1.0
Parts:
- C1, C2: footprint (none) -> Capacitor_THT:C_Radial_D6.3mm_H11.0mm_P2.50mm
- C3, C4: footprint (none) -> Capacitor_THT:C_Radial_D5.0mm_H11.0mm_P2.00mm
- D1, D2: footprint (none) -> LED_THT:LED_D5.0mm
- R100: footprint (none) -> Resistor_THT:R_Axial_DIN0207_L6.3mm_D2.5mm_P7.62mm_Horizontal
Connections:
- no-connect marks 5 -> 72
Changed lines of the file:
@@
 F 0 "C1" H 1050 4600 50  0000 L CNN
 F 1 "C 3.3uf" H 850 4500 50  0000 L CNN
-F 2 "" H 1288 4400 50  0001 C CNN
+F 2 "Capacitor_THT:C_Radial_D6.3mm_H11.0mm_P2.50mm" H 1288 4400 50  0001 C CNN
 F 3 "~" H 1250 4550 50  0001 C CNN
 	1    1250 4550
@@
 F 0 "D1" V 2489 4432 50  0000 R CNN
 F 1 "LED" V 2398 4432 50  0000 R CNN
-F 2 "" H 2450 4550 50  0001 C CNN
+F 2 "LED_THT:LED_D5.0mm" H 2450 4550 50  0001 C CNN
 F 3 "~" H 2450 4550 50  0001 C CNN
 	1    2450 4550
@@
 F 0 "R100" V 2000 4700 50  0000 C CNN
 F 1 "R" V 2100 4700 50  0000 C CNN
-F 2 "" V 2130 4700 50  0001 C CNN
+F 2 "Resistor_THT:R_Axial_DIN0207_L6.3mm_D2.5mm_P7.62mm_Horizontal" V 2130 4700 50  0001 C CNN
 F 3 "~" H 2200 4700 50  0001 C CNN
 	1    2200 4700
@@
 F 0 "C2" H 1050 5550 50  0000 L CNN
 F 1 "C 3.3uf" H 850 5450 50  0000 L CNN
-F 2 "" H 1288 5350 50  0001 C CNN
+F 2 "Capacitor_THT:C_Radial_D6.3mm_H11.0mm_P2.50mm" H 1288 5350 50  0001 C CNN
 F 3 "~" H 1250 5500 50  0001 C CNN
 	1    1250 5500
@@
 F 0 "C4" H 2065 5546 50  0000 L CNN
 F 1 "C 0.1uF" H 2065 5455 50  0000 L CNN
-F 2 "" H 1988 5350 50  0001 C CNN
+F 2 "Capacitor_THT:C_Radial_D5.0mm_H11.0mm_P2.00mm" H 1988 5350 50  0001 C CNN
 F 3 "~" H 1950 5500 50  0001 C CNN
 	1    1950 5500
@@
 F 0 "D2" V 2489 5382 50  0000 R CNN
 F 1 "LED" V 2398 5382 50  0000 R CNN
-F 2 "" H 2450 5500 50  0001 C CNN
+F 2 "LED_THT:LED_D5.0mm" H 2450 5500 50  0001 C CNN
 F 3 "~" H 2450 5500 50  0001 C CNN
 	1    2450 5500
@@
 F 0 "C3" H 2065 4596 50  0000 L CNN
 F 1 "C 0.1uF" H 2065 4505 50  0000 L CNN
-F 2 "" H 1988 4400 50  0001 C CNN
+F 2 "Capacitor_THT:C_Radial_D5.0mm_H11.0mm_P2.00mm" H 1988 4400 50  0001 C CNN
 F 3 "~" H 1950 4550 50  0001 C CNN
 	1    1950 4550
@@
 Wire Notes Line
 	4650 700  4650 1700
+NoConn ~ 10300 1450
+NoConn ~ 10300 1750
+NoConn ~ 10300 1850
+NoConn ~ 10300 1950
+NoConn ~ 10800 1450
+NoConn ~ 10800 1550
+NoConn ~ 10800 1650
+NoConn ~ 10800 1750
+NoConn ~ 10800 1850
+NoConn ~ 10800 1950
+NoConn ~ 10800 2050
+NoConn ~ 10800 2150
+NoConn ~ 10800 2250
+NoConn ~ 10800 2350
+NoConn ~ 10800 2450
+NoConn ~ 10800 2550
+NoConn ~ 10800 2650
+NoConn ~ 10800 2750
+NoConn ~ 10800 2850
+NoConn ~ 10800 2950
+NoConn ~ 10800 3050
+NoConn ~ 10800 3150
+NoConn ~ 10800 3250
+NoConn ~ 10300 3250
+NoConn ~ 10300 3150
+NoConn ~ 10300 3050
+NoConn ~ 10300 2950
+NoConn ~ 10300 2850
+NoConn ~ 10300 2750
+NoConn ~ 10300 2650
+NoConn ~ 10300 2250
+NoConn ~ 9550 1450
+NoConn ~ 9550 1550
+NoConn ~ 9550 1650
+NoConn ~ 9550 1750
+NoConn ~ 9550 1850
+NoConn ~ 9550 1950
+NoConn ~ 9550 2050
+NoConn ~ 9550 2150
+NoConn ~ 9550 2250
+NoConn ~ 9550 2350
+NoConn ~ 9550 2650
+NoConn ~ 9550 2750
+NoConn ~ 9550 2850
+NoConn ~ 9550 2950
+NoConn ~ 9550 3050
+NoConn ~ 9550 3150
+NoConn ~ 9550 3250
+NoConn ~ 9050 3250
+NoConn ~ 9050 3150
+NoConn ~ 9050 3050
+NoConn ~ 9050 2950
+NoConn ~ 9050 2850
+NoConn ~ 9050 2750
+NoConn ~ 9050 2650
+NoConn ~ 9050 2550
+NoConn ~ 9050 2450
+NoConn ~ 9050 2350
+NoConn ~ 9050 2250
+NoConn ~ 9050 2150
+NoConn ~ 9050 2050
+NoConn ~ 9050 1950
+NoConn ~ 9050 1850
+NoConn ~ 9050 1750
+NoConn ~ 9050 1650
+NoConn ~ 9050 1550
+NoConn ~ 9050 1450
 $EndSCHEMATC
