File: elec/test1/test1.kicad_pcb (KiCad board)
At the start: 2 copper layers, 70 x 59 mm, 8 parts, among them CN10 Conn_02x19_Odd_Even, CN7 Conn_02x19_Odd_Even, J1 Conn_01x04, J2 Screw_Terminal_01x02, J3 Screw_Terminal_01x02, U2 L298HN

Commit message: pcb_V1.0
Parts:
- added C1: C 3.3uf, Capacitor_THT:C_Radial_D6.3mm_H11.0mm_P2.50mm, F.Cu at (173.2, 90.0)
- added C2: C 3.3uf, Capacitor_THT:C_Radial_D6.3mm_H11.0mm_P2.50mm, F.Cu at (173.2, 99.7)
- added C3: C 0.1uF, Capacitor_THT:C_Radial_D5.0mm_H11.0mm_P2.00mm, F.Cu at (186.4, 99.2)
- added C4: C 0.1uF, Capacitor_THT:C_Radial_D5.0mm_H11.0mm_P2.00mm, F.Cu at (164.3, 99.9)
- added D1: LED, LED_THT:LED_D5.0mm, F.Cu at (154.9, 108.8)
- added D2: LED, LED_THT:LED_D5.0mm, F.Cu at (172.2, 108.8)
- added D3: 1N4007, Diode_THT:D_DO-41_SOD81_P10.16mm_Horizontal, F.Cu at (141.9, 88.0)
- added D4: 1N4007, Diode_THT:D_DO-41_SOD81_P10.16mm_Horizontal, F.Cu at (141.9, 92.3)
- added D5: 1N4007, Diode_THT:D_DO-41_SOD81_P10.16mm_Horizontal, F.Cu at (156.7, 88.0)
- added D6: 1N4007, Diode_THT:D_DO-41_SOD81_P10.16mm_Horizontal, F.Cu at (156.7, 92.3)
- added J4: Conn_01x04, Connector_JST:JST_XH_S4B-XH-A-1_1x04_P2.50mm_Horizontal, F.Cu at (181.3, 110.6)
- added J5: Conn_01x02, Connector_JST:JST_XH_S2B-XH-A_1x02_P2.50mm_Horizontal, F.Cu at (163.5, 109.1)
- added R100: R, Resistor_THT:R_Axial_DIN0207_L6.3mm_D2.5mm_P7.62mm_Horizontal, F.Cu at (181.1, 103.7)
- added U1: LM7805_TO220, Package_TO_SOT_THT:TO-220-3_Vertical, F.Cu at (182.3, 91.0)
- added U3: LP2950-3.3_TO92, Package_TO_SOT_THT:TO-92_Inline, F.Cu at (156.2, 100.2)
- moved J2 38.1 mm to (187.9, 77.6), turned to 180 degrees
- moved J3 36.5 mm to (147.3, 77.3), turned to 180 degrees
- moved U2 10.3 mm to (155.9, 83.2), turned to 0 degrees
- moved J1 0.36 mm to (141.4, 110.6)
Connections:
- CN10 pad 1: /motor_inb -> Net-(CN10-Pad1)
- CN10 pad 13: /motro_pwm -> /motor_pwm1
- CN10 pad 15: Net-(CN10-Pad15) -> /motor_pwm2
- CN10 pad 19: Net-(CN10-Pad19) -> /limit_switch
- CN10 pad 2: /motor_ina -> Net-(CN10-Pad2)
- CN10 pad 3: Net-(CN10-Pad3) -> /I2C_SCL
- CN10 pad 5: Net-(CN10-Pad5) -> /I2C_SDA
- CN7 pad 16: +3V3 -> Net-(CN7-Pad16)
- CN7 pad 18: +5V -> Net-(CN7-Pad18)
- CN7 pad 24: Net-(CN7-Pad24) -> +12V
- U2 pad 1: Net-(U2-Pad1) -> GND
- U2 pad 15: Net-(U2-Pad15) -> GND
- U2 pad 5: /motor_ina -> /motor_pwm1
- U2 pad 6: /motro_pwm -> +5V
- U2 pad 7: /motor_inb -> /motor_pwm2
Routing:
- net GND: track 56.9 -> 201.3 mm
- net +5V: track 22.2 -> 116.9 mm
- net +12V: track 33.5 -> 110.5 mm
- net /motro_pwm: track 57.0 -> 0.00 mm
- net /motor_ina: track 53.4 -> 0.00 mm
- net /motor_inb: track 49.3 -> 0.00 mm
- net /I2C_SCL: track 0.00 -> 41.1 mm
- net /I2C_SDA: track 0.00 -> 37.6 mm
- net Net-(D1-Pad1): track 0.00 -> 37.0 mm
- net /limit_switch: track 0.00 -> 36.9 mm
- net /motor_pwm1: track 0.00 -> 35.9 mm
- net /motor_pwm2: track 0.00 -> 33.1 mm
- net Net-(D3-Pad2): track 36.2 -> 64.6 mm
- net +3V3: track 29.6 -> 41.4 mm
- net Net-(D5-Pad2): track 36.1 -> 41.0 mm
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Other:
- net class Default: trace_width 0.25 -> 0.75
- net class High_current: clearance 0.4 -> 0.25; trace_width 1 -> 0.75

Commit message: pcb_V1.1
Parts:
- limit switch: renamed from J5
- renumbered J1 to encoder, J4 to end-effector
Other:
- board text added: "+12V"
- board text added: "GND"
